File: hardware/thermistor-strip/thermistor-strip.kicad_sch (KiCad schematic)
At the start: 0 parts

Commit message: Add library for thermistor ribbon connectors
Parts:
- added RT1, RT2, RT3, RT4, RT5, RT6: NCU18XH103F60RB, Murata_NCU18XH103F60RB:THRMC1608X95N, symbol Murata_NCU18XH103F60RB:NCU18XH103F60RB
Connections:
- new net GND: RT1.2, RT2.2, RT3.2, RT4.2, RT5.2, RT6.2
