File: hardware/controller/controller.kicad_sch (KiCad schematic)
At the start: 31 parts, among them J1 DC_12V_IN, J2 HDD_POWER_OUT, J3 470531000, J4 470531000, J5 Conn_01x07, Q1 2N3904, Q2 2N3904, U1 TSR0.5-2450, U2 XIAO-RP2350-SMD, U3 INA228, U4 74HC4051

Commit message: Assign custom through-hole JST S7B-ZR footprint to J5
Parts:
- J5: footprint Connector_JST:JST_ZH_S7B-ZR-SM4A-TF_1x07-1MP_P1.50mm_Horizontal -> JST_ZH_S7B-ZR:JST_ZH_B7B-ZR_1x07_P1.50mm_Horizontal
Changed lines of the file:
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@@
 			)
 		)
-		(property "Footprint" "Connector_JST:JST_ZH_S7B-ZR-SM4A-TF_1x07-1MP_P1.50mm_Horizontal"
+		(property "Footprint" "JST_ZH_S7B-ZR:JST_ZH_B7B-ZR_1x07_P1.50mm_Horizontal"
 			(at 240.03 132.08 0)
 			(hide yes)

Commit message: First complete pass of routing for controller + DRC report
Parts:
- removed NT1, NT2: NetTie_2, NetTie:NetTie-2_SMD_Pad0.5mm, symbol Device:NetTie_2
Connections:
- net 12V_HDD_SENSE is gone; now on net 12V_HDD: R4.1, U3.8 (Vbus)
- net 12V_IN_SENSE is gone; now on net 12V_IN: R3.1
- net GND: now also J5.3 (Pin_3); no longer J5.5 (Pin_5)
- net TH1: now also J5.7 (Pin_7); no longer J5.1 (Pin_1)
- net TH2: now also J5.6 (Pin_6); no longer J5.2 (Pin_2)
- net TH3: now also J5.5 (Pin_5); no longer J5.3 (Pin_3)
- net TH5: now also J5.2 (Pin_2); no longer J5.6 (Pin_6)
- net TH6: now also J5.1 (Pin_1); no longer J5.7 (Pin_7)

Commit message: updated DRC
Parts:
- U2: footprint Seeed_Studio_XIAO_Series:XIAO-RP2350-SMD -> XIAO_RP2350:XIAO-RP2350-no-underside
Changed lines of the file:
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@@
 			)
 		)
-		(property "Footprint" "Seeed_Studio_XIAO_Series:XIAO-RP2350-SMD"
+		(property "Footprint" "XIAO_RP2350:XIAO-RP2350-no-underside"
 			(at 89.408 83.566 0)
 			(hide yes)
