File: hardware/fan-controller.kicad_sch (KiCad schematic)
At the start: 29 parts, among them J1 DC_12V_IN, J2 HDD_POWER_OUT, J3 470531000, J4 470531000, J5 Conn_01x07, Q1 2N3904, Q2 2N3904, U1 TSR0.5-2450, U2 XIAO-RP2350-SMD, U3 INA228, U4 74HC4051

Commit message: Consolidate KiCad controller project and project-local FanController libraries
Parts:
- J1: footprint 54-00286:TENSILITY_54-00286 -> FanController:TENSILITY_54-00286; symbol 54-00286:54-00286 -> FanController:54-00286
- J3, J4: footprint Molex_470531000:CONN_SD-47053-001_H10p00_MOL -> FanController:CONN_SD-47053-001_H10p00_MOL; symbol Molex_470531000:470531000 -> FanController:470531000
- J5: footprint JST_ZH_S7B-ZR:JST_ZH_B7B-ZR_1x07_P1.50mm_Horizontal -> FanController:JST_ZH_B7B-ZR_1x07_P1.50mm_Horizontal
- RSH1: footprint CRF2512_FZ_R001ELF:RESC6432X80N -> FanController:RESC6432X80N; symbol CRF2512-FZ-R001ELF:CRF2512-FZ-R001ELF -> FanController:CRF2512-FZ-R001ELF
- TH7, TH8: footprint Murata_NCU18XH103F60RB:THRMC1608X95N -> FanController:THRMC1608X95N; symbol Murata_NCU18XH103F60RB:NCU18XH103F60RB -> FanController:NCU18XH103F60RB
- U2: footprint XIAO_RP2350:XIAO-RP2350-no-underside -> FanController:XIAO-RP2350-no-underside; symbol Seeed_Studio_XIAO_Series:XIAO-RP2350-SMD -> FanController:XIAO-RP2350-SMD

Commit message: Align FanController 3D model names and repair KiCad footprint references
Parts:
- U2: symbol FanController:XIAO-RP2350-SMD -> FanController:XIAO-RP2350-no-underside
Changed lines of the file:
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@@
 	)
 	(symbol
-		(lib_id "FanController:XIAO-RP2350-SMD")
+		(lib_id "FanController:XIAO-RP2350-no-underside")
 		(at 88.9 93.98 0)
 		(unit 1)
