File: hardware/fan-controller.kicad_pcb (KiCad board)
At the start: 2 copper layers, 30 x 100 mm, 33 parts, among them J1 DC_12V_IN, J2 HDD_POWER_OUT, J3 470531000, J4 470531000, J5 Conn_01x07, Q1 2N3904, Q2 2N3904, U1 TSR0.5-2450, U2 XIAO-RP2350-no-underside, U3 INA228, U4 74HC4051

Commit message: pcb trace update
Parts:
- removed J5: Conn_01x07, FanController:JST_ZH_B7B-ZR_1x07_P1.50mm_Horizontal
- removed TH8: NCU18XH103F60RB, FanController:THRMC1608X95N
- removed U4: 74HC4051, Package_SO:SOIC-16_3.9x9.9mm_P1.27mm
- added C4: 100nF, Capacitor_SMD:C_0805_2012Metric, F.Cu at (77.1, 140.3)
- added R12: 33K, Resistor_SMD:R_0805_2012Metric, F.Cu at (79.5, 136.4)
- added S1: SLW-883935-2A-D, FanController:SW_SLW-883935-2A-D, F.Cu at (66.8, 80.3)
- added TH2: NCU18XH103F60RB, FanController:THRMC1608X95N, F.Cu at (79.2, 140.3)
- R11: value 10K -> 33K
- U2: value XIAO-RP2350-no-underside -> XIAO-RP2350-SMD
- moved R11 81.5 mm to (79.0, 61.6)
- moved C3 75.9 mm to (77.1, 57.7), turned to 90 degrees
- moved C1 9.04 mm to (56.6, 77.5), turned to -90 degrees
- moved J2 7.72 mm to (57.5, 130.9)
- moved R7 6.30 mm to (75.2, 81.1)
- moved RSH1 6.18 mm to (60.0, 120.7)
- moved R5 5.49 mm to (71.9, 85.0)
- moved J3 5.15 mm to (75.1, 92.7)
- moved Q1 5.15 mm to (76.0, 87.8)
- moved R6 5.08 mm to (71.9, 88.9)
- moved J1 4.97 mm to (59.9, 110.7), turned to 0 degrees
- moved R3 3.86 mm to (59.0, 84.8), turned to 0 degrees
- moved U1 3.51 mm to (61.6, 99.0)
- moved D1 2.91 mm to (64.7, 86.9)
- moved R2 1.56 mm to (56.6, 73.7)
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- renumbered TH7 to TH1
Connections:
- C3 pad 1: +3.3V -> /TH1_ADC
- D1 pad 1: +5V -> Net-(D1-K)
- R11 pad 2: /NTC_ADC -> /TH1_ADC
- TH1 pad 1: /TH7 -> /TH1_ADC
- U2 pad 1: unconnected-(U2-D0-Pad1) -> /TH1_ADC
- U2 pad 2: /NTC_ADC -> /TH2_ADC
- U2 pad 3: /NTC_SEL2 -> unconnected-(U2-D2-Pad3)
- U2 pad 4: /NTC_SEL1 -> unconnected-(U2-D3-Pad4)
- U2 pad 7: /NTC_SEL0 -> unconnected-(U2-D6-Pad7)
Routing:
- net /TH2_ADC: track 0.00 -> 117.0 mm
- net /NTC_SEL2: track 98.3 -> 0.00 mm
- net /NTC_ADC: track 97.6 -> 0.00 mm
- net /TH7: track 96.9 -> 0.00 mm
- net /NTC_SEL1: track 93.1 -> 0.00 mm
- net /NTC_SEL0: track 83.0 -> 0.00 mm
- net GND: track 421.4 -> 372.0 mm, vias 0 -> 1
- net /TH1_ADC: track 0.00 -> 30.2 mm, vias 0 -> 2
- net +3.3V: track 152.8 -> 126.6 mm, vias 2 -> 3
- net /TH8: track 23.3 -> 0.00 mm
- net /TH6: track 21.5 -> 0.00 mm
- net /TH5: track 17.9 -> 0.00 mm
- net /12V_HDD: track 51.3 -> 65.4 mm
- net /12V_IN: track 77.9 -> 90.5 mm
- net +5V: track 39.0 -> 29.0 mm
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
Commit message: Run DRC
Parts:
- moved R5 0.27 mm to (71.9, 84.8)
Routing:
- net /12V_IN: track 90.5 -> 116.4 mm
- net /12V_HDD: track 65.4 -> 67.8 mm
- net Net-(Q1-B): track 5.72 -> 6.73 mm

Commit message: add parts to library
Parts:
- moved D1 0.60 mm to (64.7, 87.5)
- moved J3 0.12 mm to (75.0, 92.7)
Routing:
- net +3.3V: track 126.6 -> 135.5 mm
- net Net-(Q2-B): track 2.16 -> 6.58 mm
- net /12V_HDD: track 67.8 -> 65.0 mm
- net /FAN2_PWM: track 64.1 -> 63.4 mm
- net Net-(D1-K): track 6.03 -> 6.65 mm
- net Net-(D1-A): track 7.02 -> 6.40 mm
- net /TH1_ADC: track 30.2 -> 29.7 mm
